Commit message: Added initial Nav2 configuration with working AMCL

File: src/robot_description/urdf/mobile_base.xacro (robot description, xacro)
@@ -1,9 +1,9 @@
 <?xml version="1.0"?>
 <robot xmlns:xacro="http://www.ros.org/wiki/xacro">
-    <xacro:property name="car_hight" value="2.85" />
-    <xacro:property name="car_width" value="2.56" />
-    <xacro:property name="car_length" value="6.58" />
-    <xacro:property name="wheel_radius" value="0.52" />
-    <xacro:property name="wheel_length" value="0.3" />
+    <xacro:property name="car_hight" value="0.3" />
+    <xacro:property name="car_width" value="0.8" />
+    <xacro:property name="car_length" value="1.0" />
+    <xacro:property name="wheel_radius" value="0.2" />
+    <xacro:property name="wheel_length" value="0.1" />
     <xacro:macro name="wheel_inertia" params="m r h o_xyz o_rpy">
         <inertial>
@@ -32,4 +32,48 @@
         </inertial>
     </xacro:macro>
+    <link name="lidar_link">
+        <visual>
+            <geometry>
+                <cylinder radius="0.05" length="0.04"/>
+            </geometry>
+            <material name="black">
+                <color rgba="0 0 0 1"/>
+            </material>
+        </visual>
+        <collision>
+            <geometry>
+                <cylinder radius="0.05" length="0.04"/>
+            </geometry>
+        </collision>
+        <inertial>
+            <mass value="0.1"/>
+            <inertia ixx="0.0001" ixy="0" ixz="0" iyy="0.0001" iyz="0" izz="0.0001"/>
+        </inertial>
+    </link>
+    <joint name="lidar_joint" type="fixed">
+    <parent link="base_link"/> <child link="lidar_link"/>
+    <origin xyz="0 0 ${car_hight/2 + 0.02}" rpy="0 0 0"/> </joint>
+    <link name="imu_link">
+        <visual>
+            <geometry>
+                <box size="0.02 0.02 0.02"/>
+            </geometry>
+            <material name="black"/>
+        </visual>
+        <collision>
+            <geometry>
+                <box size="0.02 0.02 0.02"/>
+            </geometry>
+        </collision>
+        <inertial>
+            <mass value="0.01"/>
+            <inertia ixx="0.0001" ixy="0" ixz="0" iyy="0.0001" iyz="0" izz="0.0001"/>
+        </inertial>
+    </link>
+    <joint name="imu_joint" type="fixed">
+        <parent link="base_link"/>
+        <child link="imu_link"/>
+        <origin xyz="0 0 0.1" rpy="0 0 0"/> \
+    </joint>
     <link name="base_footprint" />
     <link name="base_link">
@@ -50,5 +94,5 @@
              <origin xyz="0 0 0" rpy="0 0 0" />
         </collision>
-        <xacro:box_inertia m="1000" x="${car_length}" y="${car_width}"
+        <xacro:box_inertia m="5" x="${car_length}" y="${car_width}"
                            z="${car_hight}" o_xyz="0 0 0" o_rpy="0 0 0" />
     </link>
@@ -68,5 +112,5 @@
              <origin xyz="0 0 0" rpy="0 0 0" />
         </collision>
-        <xacro:box_inertia m="0.01" x="0.15" y="0.3"
+        <xacro:box_inertia m="0.001" x="0.15" y="0.3"
                            z="0.08" o_xyz="0 0 0" o_rpy="0 0 0" />
     </link>
@@ -90,5 +134,5 @@
             <origin xyz="0 0 0" rpy="${pi / 2.0} 0 0" />
         </collision>
-        <xacro:wheel_inertia m="80" r="${wheel_radius}" h="${wheel_length}"
+        <xacro:wheel_inertia m="0.05" r="${wheel_radius}" h="${wheel_length}"
                              o_xyz="0 0 0" o_rpy="${pi / 2.0} 0 0" />
         </link>
@@ -138,5 +182,5 @@
         <parent link="base_link"/>
         <child link="camera_link"/>
-        <origin xyz="${(car_length + 0.15)/2} 0 ${car_hight/2 }" rpy="0 0 0"/>
+        <origin xyz="${(car_length + 0.15)/2} 0 ${car_hight/2 - 0.05}" rpy="0 0 0"/>
     </joint>
     <joint name="camera_optical_joint" type="fixed">

File: src/robot_description/urdf/mobile_base_gazebo.xacro (robot description, xacro)
@@ -2,18 +2,18 @@
 <robot xmlns:xacro="http://www.ros.org/wiki/xacro">
     <gazebo reference="base_left_front_wheel_joint">
-        <mu1 value="0.1"/>
-        <mu2 value="0.1"/>
+        <mu1 value="0.8"/>
+        <mu2 value="0.8"/>
     </gazebo>
     <gazebo reference="base_left_rear_wheel_joint">
-        <mu1 value="0.1"/>
-        <mu2 value="0.1"/>
+        <mu1 value="0.8"/>
+        <mu2 value="0.8"/>
     </gazebo>
     <gazebo reference="base_right_front_wheel_joint">
-        <mu1 value="0.1"/>
-        <mu2 value="0.1"/>
+        <mu1 value="0.8"/>
+        <mu2 value="0.8"/>
     </gazebo>
     <gazebo reference="base_right_rear_wheel_joint">
-        <mu1 value="0.1"/>
-        <mu2 value="0.1"/>
+        <mu1 value="0.8"/>
+        <mu2 value="0.8"/>
     </gazebo>
     <gazebo>
@@ -86,3 +86,34 @@
         </sensor>
     </gazebo>
+    <gazebo reference="lidar_link">
+        <sensor name="lidar" type="gpu_lidar">
+            <pose>0 0 0 0 0 0</pose>
+            <always_on>true</always_on>
+            <visualize>true</visualize> <update_rate>120</update_rate>
+            <topic>scan</topic>
+            <gz_frame_id>lidar_link</gz_frame_id>
+            <ray>
+                <scan>
+                    <horizontal>
+                        <samples>360</samples> <resolution>1</resolution>
+                        <min_angle>-3.14159</min_angle> <max_angle>3.14159</max_angle>  </horizontal>
+                </scan>
+                <range>
+                    <min>0.10</min>
+                    <max>20.0</max> <resolution>0.01</resolution>
+                </range>
+                <noise>
+                    <type>gaussian</type>
+                    <mean>0.0</mean>
+                    <stddev>0.01</stddev>
+                </noise>
+            </ray>
+        </sensor>
+    </gazebo>
+        <gazebo reference="imu_link">
+            <sensor name="imu_sensor" type="imu">
+                <always_on>1</always_on>
+                <update_rate>50</update_rate> <visualize>true</visualize>
+                <topic>/imu</topic> <gz_frame_id>imu_link</gz_frame_id> </sensor>
+        </gazebo>
 </robot>

Commit message: Latest project update.
Autonomous driving with lidar and nav2 in gazebo.

File: src/robot_description/urdf/mobile_base.xacro (robot description, xacro)
@@ -67,5 +67,5 @@
         </collision>
         <inertial>
-            <mass value="0.01"/>
+            <mass value="0.1"/>
             <inertia ixx="0.0001" ixy="0" ixz="0" iyy="0.0001" iyz="0" izz="0.0001"/>
         </inertial>
@@ -134,5 +134,5 @@
             <origin xyz="0 0 0" rpy="${pi / 2.0} 0 0" />
         </collision>
-        <xacro:wheel_inertia m="0.05" r="${wheel_radius}" h="${wheel_length}"
+        <xacro:wheel_inertia m="0.5" r="${wheel_radius}" h="${wheel_length}"
                              o_xyz="0 0 0" o_rpy="${pi / 2.0} 0 0" />
         </link>

File: src/robot_description/urdf/mobile_base_gazebo.xacro (robot description, xacro)
@@ -1,19 +1,27 @@
 <?xml version="1.0"?>
 <robot xmlns:xacro="http://www.ros.org/wiki/xacro">
-    <gazebo reference="base_left_front_wheel_joint">
-        <mu1 value="0.8"/>
-        <mu2 value="0.8"/>
-    </gazebo>
-    <gazebo reference="base_left_rear_wheel_joint">
-        <mu1 value="0.8"/>
-        <mu2 value="0.8"/>
-    </gazebo>
-    <gazebo reference="base_right_front_wheel_joint">
-        <mu1 value="0.8"/>
-        <mu2 value="0.8"/>
-    </gazebo>
-    <gazebo reference="base_right_rear_wheel_joint">
-        <mu1 value="0.8"/>
-        <mu2 value="0.8"/>
+    <gazebo reference="left_front_wheel_link">
+        <mu1>2.0</mu1>
+        <mu2>2.0</mu2>
+        <kp>10000000.0</kp>
+        <kd>1.0</kd>
+    </gazebo>
+    <gazebo reference="left_rear_wheel_link">
+        <mu1>2.0</mu1>
+        <mu2>2.0</mu2>
+        <kp>10000000.0</kp>
+        <kd>1.0</kd>
+    </gazebo>
+    <gazebo reference="right_front_wheel_link">
+        <mu1>2.0</mu1>
+        <mu2>2.0</mu2>
+        <kp>10000000.0</kp>
+        <kd>1.0</kd>
+    </gazebo>
+    <gazebo reference="right_rear_wheel_link">
+        <mu1>2.0</mu1>
+        <mu2>2.0</mu2>
+        <kp>10000000.0</kp>
+        <kd>1.0</kd>
     </gazebo>
     <gazebo>
@@ -28,4 +36,6 @@
                 <frame_id>odom</frame_id>
                 <child_frame_id>base_footprint</child_frame_id>
+                <publish_odom_tf>false</publish_odom_tf>
+                <publish_wheel_tf>false</publish_wheel_tf>
         </plugin>
     </gazebo>
@@ -37,4 +47,5 @@
                 <joint_name>base_right_front_wheel_joint</joint_name>
                 <joint_name>base_right_rear_wheel_joint</joint_name>
+                <param name="use_sim_time" value="true"/>
         </plugin>
     </gazebo>
@@ -46,5 +57,5 @@
                 <image>
                     <width>640</width>
-                    <height>480</height>
+                    <height>360</height>
                     <format>R8G8B8</format>
                 </image>
@@ -58,12 +69,20 @@
                     <stddev>0.007</stddev>
                 </noise>
+                <distortion>
+                    <k1>0.1</k1>
+                    <k2>0.1</k2>
+                    <k3>0.1</k3>
+                    <p1>0.1</p1>
+                    <p2>0.1</p2>
+                    <center>0.5 0.5</center>
+                </distortion>
                 <camera_info_topic>camera/camera_info</camera_info_topic>
             </camera>
             <always_on>1</always_on>
-            <update_rate>20</update_rate>
+            <update_rate>30</update_rate>
             <visualize>true</visualize>
             <topic>camera/image_raw</topic>
         </sensor>
-        <sensor name="rs_depth" type="depth_camera">
+         <sensor name="rs_depth" type="depth_camera">
             <always_on>true</always_on>
             <update_rate>30</update_rate>
@@ -111,9 +130,72 @@
         </sensor>
     </gazebo>
+    <gazebo>
+            <plugin filename="gz-sim-imu-system"
+                    name="gz::sim::systems::Imu">
+            </plugin>
+        </gazebo>
         <gazebo reference="imu_link">
             <sensor name="imu_sensor" type="imu">
                 <always_on>1</always_on>
-                <update_rate>50</update_rate> <visualize>true</visualize>
-                <topic>/imu</topic> <gz_frame_id>imu_link</gz_frame_id> </sensor>
+                <update_rate>200</update_rate>
+                <visualize>true</visualize>
+                <topic>/imu</topic>
+                <gz_frame_id>imu_link</gz_frame_id>
+                <imu>
+                    <angular_velocity>
+                        <x>
+                            <noise type="gaussian">
+                                <mean>0.0</mean>
+                                <stddev>0.0002</stddev> </noise>
+                        </x>
+                        <y>
+                            <noise type="gaussian">
+                                <mean>0.0</mean>
+                                <stddev>0.0002</stddev>
+                            </noise>
+                        </y>
+                        <z>
+                            <noise type="gaussian">
+                                <mean>0.0</mean>
+                                <stddev>0.0002</stddev>
+                            </noise>
+                        </z>
+                    </angular_velocity>
+                    <linear_acceleration>
+                        <x>
+                            <noise type="gaussian">
+                                <mean>0.0</mean>
+                                <stddev>0.007</stddev>
+                            </noise>
+                        </x>
+                        <y>
+                            <noise type="gaussian">
+                                <mean>0.0</mean>
+                                <stddev>0.007</stddev>
+                            </noise>
+                        </y>
+                        <z>
+                            <noise type="gaussian">
+                                <mean>0.0</mean>
+                                <stddev>0.007</stddev>
+                            </noise>
+                        </z>
+                    </linear_acceleration>
+                </imu>
+            </sensor>
         </gazebo>
+        <!--<gazebo>
+            <plugin filename="gz-sim-imu-system"
+                    name="gz::sim::systems::Imu">
+            </plugin>
+        </gazebo>
+        <gazebo reference="imu_link">
+            <sensor name="imu_sensor" type="imu">
+                <always_on>1</always_on>
+                <update_rate>300</update_rate>
+                <visualize>true</visualize>
+                <topic>/imu</topic>
+                <gz_frame_id>imu_link</gz_frame_id>
+            </sensor>
+        </gazebo> -->
 </robot>
